Commit message: update images

File: ros2_ws/src/scara_robot/urdf/scara.xacro (robot description, xacro)
@@ -7,8 +7,8 @@
   <xacro:property name="Z1" value="0.11"/>
   <xacro:property name="L2" value="0.5"/>
-  <xacro:property name="Z2" value="0.45"/>
-  <xacro:property name="H3_max" value="0.2"/>
-  <xacro:property name="H3_fixed" value="0.2"/>
-  <xacro:property name="L4" value="0.2"/>
+  <xacro:property name="Z2" value="0.4"/>
+  <xacro:property name="H3_max" value="-0.4"/>
+  <xacro:property name="H3_fixed" value="0.1"/>
+  <xacro:property name="L4" value="0.6"/>
   <xacro:property name="L5" value="1"/>
   <xacro:property name="L6" value="0.35"/>
@@ -189,5 +189,5 @@
     <origin xyz="0 0 ${-Z2}" rpy="0 0 0"/>
     <axis xyz="0 0 -1"/>
-    <limit effort="1" velocity="0.5" lower="-0.1" upper="${H3_max}"/>
+    <limit effort="1" velocity="0.5" lower="${H3_max}" upper="0.0"/>
   </joint>
   <link name="link_4">
@@ -213,11 +213,11 @@
   <link name="tcp">
     <visual>
-      <geometry><sphere radius="0.04"/></geometry>
-      <material name="gray"/>
+      <geometry><sphere radius="0.025"/></geometry>
+      <material name="celeste"/>
     </visual>
     <xacro:axis_marker xyz="0 0 0"/>
     <collision>
-      <geometry><sphere radius="0.04"/></geometry>
-      <material name="gray"/>
+      <geometry><sphere radius="0.025"/></geometry>
+      <material name="celeste"/>
     </collision>
   </link>
